Commit message: feat: Update robot materials and add color mapping functionality

File: src/robot_arm_description/urdf/materials.xacro (robot description, xacro)
@@ -1,6 +1,12 @@
 <?xml version="1.0" ?>
 <robot name="robotic_arm" xmlns:xacro="http://www.ros.org/wiki/xacro" >
-<material name="silver">
-  <color rgba="0.700 0.700 0.700 1.000"/>
+<material name="orange">
+  <color rgba="1.0 0.42 0.04 1.0"/>
+</material>
+<material name="dark_grey">
+  <color rgba="0.2 0.2 0.2 1.0"/>
+</material>
+<material name="black">
+  <color rgba="0.05 0.05 0.05 1.0"/>
 </material>
 </robot>

File: src/robot_arm_description/urdf/robotic_arm.xacro (robot description, xacro)
@@ -25,5 +25,5 @@
       <mesh filename="package://robotic_arm_description/meshes/base_link.stl" scale="0.001 0.001 0.001"/>
     </geometry>
-    <material name="silver"/>
+    <material name="dark_grey"/>
   </visual>
   <collision>
@@ -45,5 +45,5 @@
       <mesh filename="package://robotic_arm_description/meshes/link_1_1.stl" scale="0.001 0.001 0.001"/>
     </geometry>
-    <material name="silver"/>
+    <material name="orange"/>
   </visual>
   <collision>
@@ -65,5 +65,5 @@
       <mesh filename="package://robotic_arm_description/meshes/link_2_1.stl" scale="0.001 0.001 0.001"/>
     </geometry>
-    <material name="silver"/>
+    <material name="orange"/>
   </visual>
   <collision>
@@ -85,5 +85,5 @@
       <mesh filename="package://robotic_arm_description/meshes/link_3_1.stl" scale="0.001 0.001 0.001"/>
     </geometry>
-    <material name="silver"/>
+    <material name="orange"/>
   </visual>
   <collision>
@@ -105,5 +105,5 @@
       <mesh filename="package://robotic_arm_description/meshes/link_4_1.stl" scale="0.001 0.001 0.001"/>
     </geometry>
-    <material name="silver"/>
+    <material name="dark_grey"/>
   </visual>
   <collision>
@@ -125,5 +125,5 @@
       <mesh filename="package://robotic_arm_description/meshes/link_5_1.stl" scale="0.001 0.001 0.001"/>
     </geometry>
-    <material name="silver"/>
+    <material name="dark_grey"/>
   </visual>
   <collision>
@@ -151,5 +151,5 @@
       <mesh filename="package://robotic_arm_description/meshes/Gripper_Link_v1__1__1.stl" scale="0.001 0.001 0.001"/>
     </geometry>
-    <material name="silver"/>
+    <material name="black"/>
   </visual>
   <collision>
@@ -177,5 +177,5 @@
       <mesh filename="package://robotic_arm_description/meshes/Gripper_Link_v1_1.stl" scale="0.001 0.001 0.001"/>
     </geometry>
-    <material name="silver"/>
+    <material name="black"/>
   </visual>
   <collision>
@@ -197,5 +197,5 @@
       <mesh filename="package://robotic_arm_description/meshes/GripperFinger_1.stl" scale="0.001 0.001 0.001"/>
     </geometry>
-    <material name="silver"/>
+    <material name="black"/>
   </visual>
   <collision>
@@ -217,5 +217,5 @@
       <mesh filename="package://robotic_arm_description/meshes/GripperFinger2_1.stl" scale="0.001 0.001 0.001"/>
     </geometry>
-    <material name="silver"/>
+    <material name="black"/>
   </visual>
   <collision>
@@ -237,5 +237,5 @@
       <mesh filename="package://robotic_arm_description/meshes/gripper_link_gear1_v1_1.stl" scale="0.001 0.001 0.001"/>
     </geometry>
-    <material name="silver"/>
+    <material name="black"/>
   </visual>
   <collision>
