Commit message: Add robot arm control, vision system, and clean up repo

File: src/robot_arm_description/urdf/camera.xacro (robot description, xacro)
@@ -23,5 +23,5 @@
     <parent link="world"/>
     <child link="camera_link"/>
-    <origin xyz="0.0 0.5 0.5" rpy="0 1.5708 1.5708"/> <!-- Look straight down from above the workspace -->
+    <origin xyz="0.25 0.0 0.8" rpy="0 1.5708 0"/> <!-- Look straight down from above the workspace -->
   </joint>
   <!-- Gazebo Sensor -->

File: src/robot_arm_moveit2/config/robotic_arm.ros2_control.xacro (robot description, xacro)
@@ -5,6 +5,8 @@
         <ros2_control name="${name}" type="system">
             <hardware>
-                <!-- By default, set up controllers for simulation. This won't work on real hardware -->
-                <plugin>mock_components/GenericSystem</plugin>
+                <!-- Connects MoveIt 2 directly to the ESP32 Hardware Interface -->
+                <plugin>robot_arm_hardware/RobotArmSystemHardware</plugin>
+                <param name="port">/dev/ttyUSB0</param>
+                <param name="baud_rate">115200</param>
             </hardware>
             <joint name="link_1">
@@ -13,5 +15,4 @@
                   <param name="initial_value">${initial_positions['link_1']}</param>
                 </state_interface>
-                <state_interface name="velocity"/>
             </joint>
             <joint name="link_2">
@@ -20,5 +21,4 @@
                   <param name="initial_value">${initial_positions['link_2']}</param>
                 </state_interface>
-                <state_interface name="velocity"/>
             </joint>
             <joint name="link_3">
@@ -27,5 +27,4 @@
                   <param name="initial_value">${initial_positions['link_3']}</param>
                 </state_interface>
-                <state_interface name="velocity"/>
             </joint>
             <joint name="link_4">
@@ -34,5 +33,4 @@
                   <param name="initial_value">${initial_positions['link_4']}</param>
                 </state_interface>
-                <state_interface name="velocity"/>
             </joint>
             <joint name="link_5">
@@ -41,5 +39,4 @@
                   <param name="initial_value">${initial_positions['link_5']}</param>
                 </state_interface>
-                <state_interface name="velocity"/>
             </joint>
             <joint name="link_6">
@@ -48,5 +45,4 @@
                   <param name="initial_value">${initial_positions['link_6']}</param>
                 </state_interface>
-                <state_interface name="velocity"/>
             </joint>
         </ros2_control>
