Commit message: things accomplished 1. working of both thr gazebo and rviz 2. implmenting along with the moveit2 and succesfull making it move onto the next phase of the computervision control

File: src/robot_arm_description/urdf/robotic_arm.xacro (robot description, xacro)
@@ -8,4 +8,10 @@
   <xacro:include filename="$(find robotic_arm_description)/urdf/robotic_arm.gazebo" />
 </xacro:if>
+<link name="world"/>
+<joint name="world_fixed" type="fixed">
+  <origin xyz="0 0 0" rpy="0 0 0"/>
+  <parent link="world"/>
+  <child link="base_link"/>
+</joint>
 <link name="base_link">
   <inertial>

File: src/robot_arm_moveit2/config/robotic_arm.urdf.xacro (robot description, xacro)
@@ -6,4 +6,7 @@
     <!-- Import control_xacro -->
     <xacro:include filename="robotic_arm.ros2_control.xacro" />
-    <xacro:robotic_arm_ros2_control name="FakeSystem" initial_positions_file="$(arg initial_positions_file)"/>
+    <xacro:arg name="use_fake_hardware" default="true"/>
+    <xacro:if value="$(arg use_fake_hardware)">
+        <xacro:robotic_arm_ros2_control name="FakeSystem" initial_positions_file="$(arg initial_positions_file)"/>
+    </xacro:if>
 </robot>

Commit message: feat: Implement gesture control for robotic arm using MediaPipe and OpenCV
1. trying with the 21 point case , gripper not working
2. trail on giving target point and making it move based on the motion, which is causing to bring unstable need to rework on it ,

File: src/robot_arm_description/urdf/robotic_arm.xacro (robot description, xacro)
@@ -8,10 +8,4 @@
   <xacro:include filename="$(find robotic_arm_description)/urdf/robotic_arm.gazebo" />
 </xacro:if>
-<link name="world"/>
-<joint name="world_fixed" type="fixed">
-  <origin xyz="0 0 0" rpy="0 0 0"/>
-  <parent link="world"/>
-  <child link="base_link"/>
-</joint>
 <link name="base_link">
   <inertial>
@@ -25,5 +19,5 @@
       <mesh filename="package://robotic_arm_description/meshes/base_link.stl" scale="0.001 0.001 0.001"/>
     </geometry>
-    <material name="dark_grey"/>
+    <material name="silver"/>
   </visual>
   <collision>
@@ -45,5 +39,5 @@
       <mesh filename="package://robotic_arm_description/meshes/link_1_1.stl" scale="0.001 0.001 0.001"/>
     </geometry>
-    <material name="orange"/>
+    <material name="silver"/>
   </visual>
   <collision>
@@ -65,5 +59,5 @@
       <mesh filename="package://robotic_arm_description/meshes/link_2_1.stl" scale="0.001 0.001 0.001"/>
     </geometry>
-    <material name="orange"/>
+    <material name="silver"/>
   </visual>
   <collision>
@@ -85,5 +79,5 @@
       <mesh filename="package://robotic_arm_description/meshes/link_3_1.stl" scale="0.001 0.001 0.001"/>
     </geometry>
-    <material name="orange"/>
+    <material name="silver"/>
   </visual>
   <collision>
@@ -105,5 +99,5 @@
       <mesh filename="package://robotic_arm_description/meshes/link_4_1.stl" scale="0.001 0.001 0.001"/>
     </geometry>
-    <material name="dark_grey"/>
+    <material name="silver"/>
   </visual>
   <collision>
@@ -125,5 +119,5 @@
       <mesh filename="package://robotic_arm_description/meshes/link_5_1.stl" scale="0.001 0.001 0.001"/>
     </geometry>
-    <material name="dark_grey"/>
+    <material name="silver"/>
   </visual>
   <collision>
@@ -151,5 +145,5 @@
       <mesh filename="package://robotic_arm_description/meshes/Gripper_Link_v1__1__1.stl" scale="0.001 0.001 0.001"/>
     </geometry>
-    <material name="black"/>
+    <material name="silver"/>
   </visual>
   <collision>
@@ -177,5 +171,5 @@
       <mesh filename="package://robotic_arm_description/meshes/Gripper_Link_v1_1.stl" scale="0.001 0.001 0.001"/>
     </geometry>
-    <material name="black"/>
+    <material name="silver"/>
   </visual>
   <collision>
@@ -197,5 +191,5 @@
       <mesh filename="package://robotic_arm_description/meshes/GripperFinger_1.stl" scale="0.001 0.001 0.001"/>
     </geometry>
-    <material name="black"/>
+    <material name="silver"/>
   </visual>
   <collision>
@@ -217,5 +211,5 @@
       <mesh filename="package://robotic_arm_description/meshes/GripperFinger2_1.stl" scale="0.001 0.001 0.001"/>
     </geometry>
-    <material name="black"/>
+    <material name="silver"/>
   </visual>
   <collision>
@@ -237,5 +231,5 @@
       <mesh filename="package://robotic_arm_description/meshes/gripper_link_gear1_v1_1.stl" scale="0.001 0.001 0.001"/>
     </geometry>
-    <material name="black"/>
+    <material name="silver"/>
   </visual>
   <collision>

Commit message: feat: Integrate vision and hardware control for robotic arm
- Added a new camera URDF model to the robot arm description for simulation.
- Created an empty SDF world file for Gazebo simulation with necessary plugins for sensors.
- Implemented a hardware interface for controlling the robotic arm via serial communication.
- Developed a vision node using YOLO for object detection and a sorting planner node for executing pick-and-place tasks.
- Enhanced the Gazebo launch file to include the new world and camera topics for ROS-Gazebo bridge.
- Added necessary package files and configurations for the new robot_arm_hardware and robot_arm_vision packages.
- Implemented basic error handling and logging for vision processing and planning.

File: src/robot_arm_description/urdf/robotic_arm.xacro (robot description, xacro)
@@ -8,4 +8,11 @@
   <xacro:include filename="$(find robotic_arm_description)/urdf/robotic_arm.gazebo" />
 </xacro:if>
+<xacro:include filename="$(find robotic_arm_description)/urdf/camera.xacro" />
+<link name="world"/>
+<joint name="world_joint" type="fixed">
+  <parent link="world"/>
+  <child link="base_link"/>
+  <origin xyz="0 0 0" rpy="0 0 0"/>
+</joint>
 <link name="base_link">
   <inertial>
@@ -19,5 +26,5 @@
       <mesh filename="package://robotic_arm_description/meshes/base_link.stl" scale="0.001 0.001 0.001"/>
     </geometry>
-    <material name="silver"/>
+    <material name="dark_grey"/>
   </visual>
   <collision>
@@ -39,5 +46,5 @@
       <mesh filename="package://robotic_arm_description/meshes/link_1_1.stl" scale="0.001 0.001 0.001"/>
     </geometry>
-    <material name="silver"/>
+    <material name="dark_grey"/>
   </visual>
   <collision>
@@ -59,5 +66,5 @@
       <mesh filename="package://robotic_arm_description/meshes/link_2_1.stl" scale="0.001 0.001 0.001"/>
     </geometry>
-    <material name="silver"/>
+    <material name="dark_grey"/>
   </visual>
   <collision>
@@ -79,5 +86,5 @@
       <mesh filename="package://robotic_arm_description/meshes/link_3_1.stl" scale="0.001 0.001 0.001"/>
     </geometry>
-    <material name="silver"/>
+    <material name="dark_grey"/>
   </visual>
   <collision>
@@ -99,5 +106,5 @@
       <mesh filename="package://robotic_arm_description/meshes/link_4_1.stl" scale="0.001 0.001 0.001"/>
     </geometry>
-    <material name="silver"/>
+    <material name="dark_grey"/>
   </visual>
   <collision>
@@ -119,5 +126,5 @@
       <mesh filename="package://robotic_arm_description/meshes/link_5_1.stl" scale="0.001 0.001 0.001"/>
     </geometry>
-    <material name="silver"/>
+    <material name="dark_grey"/>
   </visual>
   <collision>
@@ -145,5 +152,5 @@
       <mesh filename="package://robotic_arm_description/meshes/Gripper_Link_v1__1__1.stl" scale="0.001 0.001 0.001"/>
     </geometry>
-    <material name="silver"/>
+    <material name="dark_grey"/>
   </visual>
   <collision>
@@ -171,5 +178,5 @@
       <mesh filename="package://robotic_arm_description/meshes/Gripper_Link_v1_1.stl" scale="0.001 0.001 0.001"/>
     </geometry>
-    <material name="silver"/>
+    <material name="dark_grey"/>
   </visual>
   <collision>
@@ -191,5 +198,5 @@
       <mesh filename="package://robotic_arm_description/meshes/GripperFinger_1.stl" scale="0.001 0.001 0.001"/>
     </geometry>
-    <material name="silver"/>
+    <material name="dark_grey"/>
   </visual>
   <collision>
@@ -211,5 +218,5 @@
       <mesh filename="package://robotic_arm_description/meshes/GripperFinger2_1.stl" scale="0.001 0.001 0.001"/>
     </geometry>
-    <material name="silver"/>
+    <material name="dark_grey"/>
   </visual>
   <collision>
@@ -231,5 +238,5 @@
       <mesh filename="package://robotic_arm_description/meshes/gripper_link_gear1_v1_1.stl" scale="0.001 0.001 0.001"/>
     </geometry>
-    <material name="silver"/>
+    <material name="dark_grey"/>
   </visual>
   <collision>

Commit message: Add new SDF models for red boxes and Arduino environment setup script
- Created SDF files for red box models: red_box_demo.sdf, red_box_multi_a.sdf, red_box_multi_b.sdf, red_box_multi_c.sdf
- Added Arduino environment setup script: use_pendrive_env.sh
- Introduced a new Arduino sketch for gripper limit finding: test_03_gripper_limit_finder.ino
- Updated thesis documents in DOCX format

File: src/robot_arm_description/urdf/robotic_arm.xacro (robot description, xacro)
@@ -287,5 +287,5 @@
   <child link="Gripper_Link_Gear#1_v1_1"/>
   <axis xyz="-0.0 0.0 1.0"/>
-  <limit lower="-1.0" upper="1.0" effort="10.0" velocity="0.5"/>
+  <limit lower="-1.0472" upper="0.0" effort="10.0" velocity="0.5"/>
 </joint>
 <joint name="link_10" type="continuous">
