Commit message: feat: Add comprehensive setup documentation and scripts for ESP32-CAM based autonomous sorting system
- Created START_HERE.md for a quick start guide to set up ESP32-CAM streaming.
- Added build_autonomous_sorting.sh script to automate the build process for ROS 2 packages.
- Introduced AUTONOMOUS_SORTING_QUICKSTART.md for end-to-end setup and testing instructions.
- Developed HARDWARE_AUTONOMOUS_SORTING_SETUP.md as a detailed guide for hardware setup and calibration.
- Implemented hardware_gesture.launch.py for gesture control of the robotic arm.
- Created hardware_sorting.launch.py to launch the complete autonomous sorting pipeline.
- Added esp32_camera_bridge.py to connect ESP32-CAM MJPEG stream to ROS 2 Image messages.

File: src/robot_arm_moveit2/config/robotic_arm.ros2_control.xacro (robot description, xacro)
@@ -1,5 +1,5 @@
 <?xml version="1.0"?>
 <robot xmlns:xacro="http://www.ros.org/wiki/xacro">
-    <xacro:macro name="robotic_arm_ros2_control" params="name initial_positions_file">
+    <xacro:macro name="robotic_arm_ros2_control" params="name initial_positions_file serial_port baud_rate">
         <xacro:property name="initial_positions" value="${xacro.load_yaml(initial_positions_file)['initial_positions']}"/>
         <ros2_control name="${name}" type="system">
@@ -7,6 +7,6 @@
                 <!-- Connects MoveIt 2 directly to the ESP32 Hardware Interface -->
                 <plugin>robot_arm_hardware/RobotArmSystemHardware</plugin>
-                <param name="port">/dev/ttyUSB0</param>
-                <param name="baud_rate">115200</param>
+                <param name="port">${serial_port}</param>
+                <param name="baud_rate">${baud_rate}</param>
             </hardware>
             <joint name="link_1">

File: src/robot_arm_moveit2/config/robotic_arm.urdf.xacro (robot description, xacro)
@@ -2,4 +2,6 @@
 <robot xmlns:xacro="http://www.ros.org/wiki/xacro" name="robotic_arm">
     <xacro:arg name="initial_positions_file" default="initial_positions.yaml" />
+    <xacro:arg name="serial_port" default="/dev/ttyUSB0" />
+    <xacro:arg name="baud_rate" default="115200" />
     <!-- Import robotic_arm urdf file -->
     <xacro:include filename="$(find robotic_arm_description)/urdf/robotic_arm.xacro" />
@@ -8,5 +10,9 @@
     <xacro:arg name="use_fake_hardware" default="true"/>
     <xacro:if value="$(arg use_fake_hardware)">
-        <xacro:robotic_arm_ros2_control name="FakeSystem" initial_positions_file="$(arg initial_positions_file)"/>
+        <xacro:robotic_arm_ros2_control
+            name="FakeSystem"
+            initial_positions_file="$(arg initial_positions_file)"
+            serial_port="$(arg serial_port)"
+            baud_rate="$(arg baud_rate)"/>
     </xacro:if>
 </robot>
